Commit message: ubot rviz working

File: urdf/materials.urdf.xacro (robot description, xacro)
@@ -1,29 +1,29 @@
 <?xml version="1.0"?>
 <robot>
-  <material name="youBot/Orange">
+  <material name="Orange">
     <color rgba="1.0 0.4 0.0 1.0"/>
   </material>
-  <material name="youBot/Grey">
+  <material name="Grey">
     <color rgba="0.7 0.7 0.7 1.0"/>
   </material>
-  <material name="youBot/DarkGrey">
+  <material name="DarkGrey">
     <color rgba="0.3 0.3 0.3 1.0"/>
   </material>
-  <material name="youBot/White">
+  <material name="White">
     <color rgba="1.0 1.0 1.0 1.0"/>
   </material>
-  <material name="youBot/Black">
+  <material name="Black">
     <color rgba="0.0 0.0 0.0 1.0"/>
   </material>
-  <material name="youBot/Red">
+  <material name="Red">
     <color rgba="1.0 0.0 0.0 1.0"/>
   </material>
-  <material name="youBot/Green">
+  <material name="Green">
     <color rgba="0.0 1.0 0.0 1.0"/>
   </material>
-  <material name="youBot/Blue">
+  <material name="Blue">
     <color rgba="0.0 0.0 0.8 1.0"/>
   </material>
-  <material name="youBot/LightGrey">
+  <material name="LightGrey">
     <color rgba="0.82 0.82 0.82 1.0"/>
   </material>

File: urdf/youbot.urdf.xacro (robot description, xacro)
@@ -7,19 +7,15 @@
   <!-- The following xacro:included files set up definitions of parts of the robot body -->
   <!-- misc common stuff? -->
-  <xacro:include filename="$(find youbot_description)/urdf/common.xacro" />
+  <xacro:include filename="$(find youbot_gz)/urdf/common.xacro" />
   <!-- youbot base -->
-  <xacro:include filename="$(find youbot_description)/urdf/youbot_base/base.urdf.xacro" />
+  <xacro:include filename="$(find youbot_gz)/urdf/youbot_base/base.urdf.xacro" />
   <!-- youbot plate -->
-  <xacro:include filename="$(find youbot_description)/urdf/youbot_plate/plate.urdf.xacro" />
+  <xacro:include filename="$(find youbot_gz)/urdf/youbot_plate/plate.urdf.xacro" />
   <!-- youbot arm -->
-  <xacro:include filename="$(find youbot_description)/urdf/youbot_arm/arm.urdf.xacro"/>
+  <xacro:include filename="$(find youbot_gz)/urdf/youbot_arm/arm.urdf.xacro"/>
   <!-- youbot gripper -->
-  <xacro:include filename="$(find youbot_description)/urdf/youbot_gripper/gripper.urdf.xacro" />
-  <!-- controller manager -->
-  <xacro:include filename="$(find youbot_description)/controller/ros_controller.urdf.xacro" />
+  <xacro:include filename="$(find youbot_gz)/urdf/youbot_gripper/gripper.urdf.xacro" />
   <!-- materials for visualization -->
-  <xacro:include filename="$(find youbot_description)/urdf/materials.urdf.xacro" />
-  <!-- sensors -->
-  <xacro:include filename="$(find youbot_description)/urdf/sensors/hokuyo_urg04_laser.urdf.xacro"/>
+  <xacro:include filename="$(find youbot_gz)/urdf/materials.urdf.xacro" />
   <!-- Now we can start using the macros xacro:included above to define the actual youbot -->
   <!-- The first use of a macro.  This one was defined in base.urdf.xacro above.
@@ -42,6 +38,7 @@
   </xacro:youbot_gripper>
   <!-- base laser front -->
-  <xacro:hokuyo_urg04_laser name="base_laser_front" parent="base" ros_topic="scan_front" update_rate="10" min_angle="-1.57" max_angle="1.57">
+  <!-- <xacro:hokuyo_urg04_laser name="base_laser_front" parent="base" ros_topic="scan_front" update_rate="10" min_angle="-1.57" max_angle="1.57">
     <origin xyz="0.3 0 -0.03" rpy="0 0 0"/>
   </xacro:hokuyo_urg04_laser>
+  -->
 </robot>

File: urdf/youbot_arm/arm.urdf.xacro (robot description, xacro)
@@ -4,7 +4,7 @@
         xmlns:interface="http://playerstage.sourceforge.net/gazebo/xmlschema/#interface"
         xmlns:xacro="http://www.ros.org/wiki/xacro/#interface">
-	<xacro:include filename="$(find youbot_description)/urdf/youbot_arm/arm.gazebo.xacro" />
-	<xacro:include filename="$(find youbot_description)/urdf/youbot_arm/arm.transmission.xacro" />
-	<xacro:include filename="$(find youbot_description)/urdf/youbot_arm/limits.urdf.xacro" />
+	<xacro:include filename="$(find youbot_gz)/urdf/youbot_arm/arm.gazebo.xacro" />
+	<xacro:include filename="$(find youbot_gz)/urdf/youbot_arm/arm.transmission.xacro" />
+	<xacro:include filename="$(find youbot_gz)/urdf/youbot_arm/limits.urdf.xacro" />
 	<xacro:macro name="youbot_arm" params="parent name *origin">
 		<!-- joint between base_link and arm_0_link -->
@@ -24,7 +24,7 @@
 				<origin xyz="0 0 0" rpy="0 0 0" />
 				<geometry>
-					<mesh filename="package://youbot_description/meshes/youbot_arm/arm0.dae" />
-				</geometry>
-				<material name="youBot/DarkGrey" />
+					<mesh filename="package://youbot_gz/meshes/youbot_arm/arm0.dae" />
+				</geometry>
+				<material name="DarkGrey" />
 			</visual>
 			<collision>
@@ -32,5 +32,5 @@
 				<origin xyz="0 0 0" rpy="0 0 0"/>
 				<geometry>
-					<mesh filename="package://youbot_description/meshes/youbot_arm/arm0_convex.dae" />
+					<mesh filename="package://youbot_gz/meshes/youbot_arm/arm0_convex.dae" />
 					<!--<cylinder length="0.078" radius="0.093"/>-->
 				</geometry>
@@ -63,7 +63,7 @@
 				<origin xyz="0 0 0" rpy="0 0 0" />
 				<geometry>
-					<mesh filename="package://youbot_description/meshes/youbot_arm/arm1.dae" />
-				</geometry>
-				<material name="youBot/Orange" />
+					<mesh filename="package://youbot_gz/meshes/youbot_arm/arm1.dae" />
+				</geometry>
+				<material name="Orange" />
 			</visual>
 			<collision>
@@ -71,5 +71,5 @@
 				<origin xyz="0 0 0" rpy="0 0 0" />
 				<geometry>
-					<mesh filename="package://youbot_description/meshes/youbot_arm/arm1_convex.dae" />
+					<mesh filename="package://youbot_gz/meshes/youbot_arm/arm1_convex.dae" />
 					<!--<cylinder length="0.102" radius="0.080"/>-->
 				</geometry>
@@ -95,5 +95,5 @@
 			<origin xyz="0 -0.032 0.078" rpy="0 0 0" />
 				<geometry>
-					<mesh filename="package://youbot_description/meshes/youbot_arm/arm2.dae" />
+					<mesh filename="package://youbot_gz/meshes/youbot_arm/arm2.dae" />
 				</geometry>
 			</visual>
@@ -102,5 +102,5 @@
 				<origin xyz="0 -0.032 0.078" rpy="0 0 0" />
 				<geometry>
-					<mesh filename="package://youbot_description/meshes/youbot_arm/arm2_convex.dae" />
+					<mesh filename="package://youbot_gz/meshes/youbot_arm/arm2_convex.dae" />
 					<!--<box size="0.074 0.082 0.222"/>-->
 				</geometry>
@@ -134,7 +134,7 @@
 				<origin xyz="0.000 0.028 0.079" rpy="0 0 0" />
 				<geometry>
-					<mesh filename="package://youbot_description/meshes/youbot_arm/arm3.dae" />
-				</geometry>
-				<material name="youBot/Orange" />
+					<mesh filename="package://youbot_gz/meshes/youbot_arm/arm3.dae" />
+				</geometry>
+				<material name="Orange" />
 			</visual>
 			<collision>
@@ -142,5 +142,5 @@
 				<origin xyz="0.000 0.028 0.079" rpy="0 0 0" />
 				<geometry>
-					<mesh filename="package://youbot_description/meshes/youbot_arm/arm3_convex.dae" />
+					<mesh filename="package://youbot_gz/meshes/youbot_arm/arm3_convex.dae" />
 					<!--<box size="0.064 0.054 0.192"/>-->
 				</geometry>
@@ -166,7 +166,7 @@
 				<origin xyz="0 -0.010 0.029" rpy="0 0 0"/>
 				<geometry>
-					<mesh filename="package://youbot_description/meshes/youbot_arm/arm4.dae" />
-				</geometry>
-				<material name="youBot/Orange" />
+					<mesh filename="package://youbot_gz/meshes/youbot_arm/arm4.dae" />
+				</geometry>
+				<material name="Orange" />
 			</visual>
 			<collision>
@@ -174,5 +174,5 @@
 				<origin xyz="0 -0.010 0.029" rpy="0 0 0"/>
 				<geometry>
-					<mesh filename="package://youbot_description/meshes/youbot_arm/arm4_convex.dae" />
+					<mesh filename="package://youbot_gz/meshes/youbot_arm/arm4_convex.dae" />
 					<!--<box size="0.058 0.100 0.118"/>-->
 				</geometry>
@@ -198,12 +198,12 @@
 				<origin xyz="0.003 0 -0.034" rpy="0 0 0" />
 				<geometry>
-					<mesh filename="package://youbot_description/meshes/youbot_arm/arm5.dae" />
-				</geometry>
-				<material name="youBot/DarkGrey" />
+					<mesh filename="package://youbot_gz/meshes/youbot_arm/arm5.dae" />
+				</geometry>
+				<material name="DarkGrey" />
 			</visual>
 			<collision>
 				<origin xyz="0.003 0 -0.034" rpy="0 0 0" />
 				<geometry>
-					<mesh filename="package://youbot_description/meshes/youbot_arm/arm5_convex.dae" />
+					<mesh filename="package://youbot_gz/meshes/youbot_arm/arm5_convex.dae" />
 					<!--<box size="0.054 0.096 0.030"/>-->
 				</geometry>

File: urdf/youbot_base/base.urdf.xacro (robot description, xacro)
@@ -4,6 +4,6 @@
        xmlns:interface="http://playerstage.sourceforge.net/gazebo/xmlschema/#interface"
        xmlns:xacro="http://www.ros.org/wiki/xacro/#interface">
-  <xacro:include filename="$(find youbot_description)/urdf/youbot_base/base.gazebo.xacro"/>
-  <xacro:include filename="$(find youbot_description)/urdf/youbot_base/base.transmission.xacro"/>
+  <xacro:include filename="$(find youbot_gz)/urdf/youbot_base/base.gazebo.xacro"/>
+  <xacro:include filename="$(find youbot_gz)/urdf/youbot_base/base.transmission.xacro"/>
   <!-- simplified box collision geometry for base -->
   <xacro:property name="base_size_x" value="0.570"/>
@@ -47,7 +47,7 @@
         <origin xyz="0 0 0" rpy="0 0 0"/>
         <geometry>
-          <mesh filename="package://youbot_description/meshes/youbot_base/base.dae"/>
-        </geometry>
-        <material name="youBot/DarkGrey"/>
+          <mesh filename="package://youbot_gz/meshes/youbot_base/base.dae"/>
+        </geometry>
+        <material name="DarkGrey"/>
       </visual>
       <collision>
@@ -55,5 +55,5 @@
         <geometry>
           <!--<box size="${base_size_x} ${base_size_y} ${base_size_z}" />-->
-          <mesh filename="package://youbot_description/meshes/youbot_base/base_convex.dae"/>
+          <mesh filename="package://youbot_gz/meshes/youbot_base/base_convex.dae"/>
         </geometry>
       </collision>
@@ -93,9 +93,9 @@
       <visual>
         <origin xyz="0 0 0" rpy="0 0 0"/>
-        <!--<mesh filename="package://youbot_description/meshes/youbot_base/youbot_wheel.stl" />-->
-        <geometry>
-          <sphere radius="${wheel_radius}"/>
-        </geometry>
-        <material name="youBot/Orange"/>
+        <!--<mesh filename="package://youbot_gz/meshes/youbot_base/youbot_wheel.stl" />-->
+        <geometry>
+          <sphere radius="${wheel_radius}"/>
+        </geometry>
+        <material name="Orange"/>
       </visual>
       <collision>
@@ -141,8 +141,8 @@
         <origin xyz="0 0 0" rpy="0 0 0"/>
         <geometry>
-          <!--<mesh filename="package://youbot_description/meshes/youbot_base/youbot_wheel.stl" />-->
-          <sphere radius="${wheel_radius}"/>
-        </geometry>
-        <material name="youBot/Orange"/>
+          <!--<mesh filename="package://youbot_gz/meshes/youbot_base/youbot_wheel.stl" />-->
+          <sphere radius="${wheel_radius}"/>
+        </geometry>
+        <material name="Orange"/>
       </visual>
       <collision>
@@ -188,8 +188,8 @@
         <origin xyz="0 0 0" rpy="0 0 0"/>
         <geometry>
-          <!--<mesh filename="package://youbot_description/meshes/youbot_base/youbot_wheel.stl" />-->
-          <sphere radius="${wheel_radius}"/>
-        </geometry>
-        <material name="youBot/Orange"/>
+          <!--<mesh filename="package://youbot_gz/meshes/youbot_base/youbot_wheel.stl" />-->
+          <sphere radius="${wheel_radius}"/>
+        </geometry>
+        <material name="Orange"/>
       </visual>
       <collision>
@@ -235,8 +235,8 @@
         <origin xyz="0 0 0" rpy="0 0 0"/>
         <geometry>
-          <!--<mesh filename="package://youbot_description/meshes/youbot_base/youbot_wheel.stl" />-->
-          <sphere radius="${wheel_radius}"/>
-        </geometry>
-        <material name="youBot/Orange"/>
+          <!--<mesh filename="package://youbot_gz/meshes/youbot_base/youbot_wheel.stl" />-->
+          <sphere radius="${wheel_radius}"/>
+        </geometry>
+        <material name="Orange"/>
       </visual>
       <collision>

File: urdf/youbot_gripper/gripper.urdf.xacro (robot description, xacro)
@@ -4,7 +4,7 @@
        xmlns:interface="http://playerstage.sourceforge.net/gazebo/xmlschema/#interface"
        xmlns:xacro="http://www.ros.org/wiki/xacro/#interface">
-	<xacro:include filename="$(find youbot_description)/urdf/youbot_gripper/gripper.gazebo.xacro" />
-	<xacro:include filename="$(find youbot_description)/urdf/youbot_gripper/gripper.transmission.xacro" />
-	<xacro:include filename="$(find youbot_description)/urdf/youbot_gripper/limits.urdf.xacro" />
+	<xacro:include filename="$(find youbot_gz)/urdf/youbot_gripper/gripper.gazebo.xacro" />
+	<xacro:include filename="$(find youbot_gz)/urdf/youbot_gripper/gripper.transmission.xacro" />
+	<xacro:include filename="$(find youbot_gz)/urdf/youbot_gripper/limits.urdf.xacro" />
 	<xacro:macro name="youbot_gripper" params="parent name *origin">
 		<!-- joint between arm_7_link and sdh_palm_link -->
@@ -23,5 +23,5 @@
 				<origin xyz="0 0 0" rpy="0 0 0" />
 				<geometry>
-					<mesh filename="package://youbot_description/meshes/youbot_gripper/palm.dae" />
+					<mesh filename="package://youbot_gz/meshes/youbot_gripper/palm.dae" />
 				</geometry>
 				<material name="Black" />
@@ -31,5 +31,5 @@
 				<geometry>
 					<!--<box size="0.050 0.094 0.054"/>-->
-					<mesh filename="package://youbot_description/meshes/youbot_gripper/palm_convex.dae" />
+					<mesh filename="package://youbot_gz/meshes/youbot_gripper/palm_convex.dae" />
 				</geometry>
 			</collision>
@@ -53,5 +53,5 @@
 				<origin xyz="0 0 0" rpy="0 0 0" />
 				<geometry>
-					<mesh filename="package://youbot_description/meshes/youbot_gripper/finger.dae" />
+					<mesh filename="package://youbot_gz/meshes/youbot_gripper/finger.dae" />
 				</geometry>
 				<material name="Black" />
@@ -61,5 +61,5 @@
 				<geometry>
 					<!--<box size="0.014 0.020 0.046"/>-->
-					<mesh filename="package://youbot_description/meshes/youbot_gripper/finger_convex.dae" />
+					<mesh filename="package://youbot_gz/meshes/youbot_gripper/finger_convex.dae" />
 				</geometry>
 			</collision>
@@ -83,5 +83,5 @@
 				<origin xyz="0 0 0" rpy="0 0 0" />
 				<geometry>
-					<mesh filename="package://youbot_description/meshes/youbot_gripper/finger.dae" />
+					<mesh filename="package://youbot_gz/meshes/youbot_gripper/finger.dae" />
 				</geometry>
 				<material name="Black" />
@@ -91,5 +91,5 @@
 				<geometry>
 					<!--<box size="0.014 0.020 0.046"/>-->
-					<mesh filename="package://youbot_description/meshes/youbot_gripper/finger_convex.dae" />
+					<mesh filename="package://youbot_gz/meshes/youbot_gripper/finger_convex.dae" />
 				</geometry>
 			</collision>

File: urdf/youbot_plate/plate.urdf.xacro (robot description, xacro)
@@ -20,5 +20,5 @@
 				<origin xyz="0 0 0" rpy="0 0 0" />
 				<geometry>
-					<mesh filename="package://youbot_description/meshes/youbot_plate/plate.dae" />
+					<mesh filename="package://youbot_gz/meshes/youbot_plate/plate.dae" />
 				</geometry>
 				<material name="DarkGrey"/>
@@ -27,5 +27,5 @@
 				<origin xyz="0 0 0" rpy="0 0 0" />
 				<geometry>
-					<mesh filename="package://youbot_description/meshes/youbot_plate/plate_convex.dae" />
+					<mesh filename="package://youbot_gz/meshes/youbot_plate/plate_convex.dae" />
 				</geometry>
 			</collision>
